File: FDDuino.kicad/FDDuino.sch (KiCad schematic (older format))
At the start: 3 parts, among them P3 SPC1K-EXT, U1 8255

Commit message: Weekend works for FDDuino and MSXuino
Connections:
- net +5V: no longer SHIELD1.5V_5
- net /CS: now also SHIELD1.4; no longer SHIELD1.3
- net /RD: now also SHIELD1.5; no longer SHIELD1.4
- net /WR: now also SHIELD1.6; no longer SHIELD1.5
- net A0: now also SHIELD1.7; no longer SHIELD1.6
- net A1: now also SHIELD1.8; no longer SHIELD1.7
- net PC0: now also SHIELD1.22 (PA0); no longer SHIELD1.AD7
- net PC1: now also SHIELD1.23 (PA1); no longer SHIELD1.AD6
- net PC2: now also SHIELD1.24 (PA2); no longer SHIELD1.AD5
- net PC3: now also SHIELD1.25 (PA3); no longer SHIELD1.AD4
- net PC4: now also SHIELD1.26 (PA4); no longer SHIELD1.AD3
- net PC5: now also SHIELD1.27 (PA5); no longer SHIELD1.AD2
- net PC6: now also SHIELD1.28 (PA6); no longer SHIELD1.AD1
- net PC7: now also SHIELD1.29 (PA7); no longer SHIELD1.AD0
- net RESET: no longer SHIELD1.8
- net PA3: now reaches U1.1 (PA3)
- net PA3: now also SHIELD1.AD4; no longer SHIELD1.34 (PC3)
- net PB0: now reaches U1.18 (PB0)
- net PB0: now also SHIELD1.37 (PC0); no longer SHIELD1.29 (PA7)
- net PB1: now reaches U1.19 (PB1)
- net PB1: now also SHIELD1.36 (PC1); no longer SHIELD1.28 (PA6)
- net PA2: now reaches U1.2 (PA2)
- net PA2: now also SHIELD1.AD5; no longer SHIELD1.35 (PC2)
- net PB2: now reaches U1.20 (PB2)
- net PB2: now also SHIELD1.35 (PC2); no longer SHIELD1.27 (PA5)
- net PB3: now reaches U1.21 (PB3)
- net PB3: now also SHIELD1.34 (PC3); no longer SHIELD1.26 (PA4)
- net PB4: now reaches U1.22 (PB4)
- net PB4: now also SHIELD1.33 (PC4); no longer SHIELD1.25 (PA3)
- net PB5: now reaches U1.23 (PB5)
- net PB5: now also SHIELD1.32 (PC5); no longer SHIELD1.24 (PA2)
- net PB6: now reaches U1.24 (PB6)
- net PB6: now also SHIELD1.31 (PC6); no longer SHIELD1.23 (PA1)
- net PB7: now reaches U1.25 (PB7)
- net PB7: now also SHIELD1.30 (PC7); no longer SHIELD1.22 (PA0)
- net PA1: now reaches U1.3 (PA1)
- net PA1: now also SHIELD1.AD6; no longer SHIELD1.36 (PC1)
- net PA7: now reaches U1.37 (PA7)
- net PA7: now also SHIELD1.AD0; no longer SHIELD1.30 (PC7)
- net PA6: now reaches U1.38 (PA6)
- net PA6: now also SHIELD1.AD1; no longer SHIELD1.31 (PC6)
- net PA5: now reaches U1.39 (PA5)
- net PA5: now also SHIELD1.AD2; no longer SHIELD1.32 (PC5)
- net PA0: now reaches U1.4 (PA0)
- net PA0: now also SHIELD1.AD7; no longer SHIELD1.37 (PC0)
- net PA4: now reaches U1.40 (PA4)
- net PA4: now also SHIELD1.AD3; no longer SHIELD1.33 (PC4)
Changed lines of the file:
@@
 	1    0    0    -1
 $EndComp
-Wire Wire Line
-	6150 1600 7750 1600
-Wire Wire Line
-	6150 1700 7750 1700
-Wire Wire Line
-	6150 1800 7750 1800
-Wire Wire Line
-	6150 1900 7750 1900
-Wire Wire Line
-	6150 2000 7750 2000
-Wire Wire Line
-	6150 2100 7750 2100
-Wire Wire Line
-	6150 2200 7750 2200
-Wire Wire Line
-	6150 2400 7750 2400
-Wire Wire Line
-	6150 2500 7750 2500
-Wire Wire Line
-	6150 2600 7750 2600
-Wire Wire Line
-	6150 2700 7750 2700
-Wire Wire Line
-	6150 2800 7750 2800
-Wire Wire Line
-	6150 2900 7750 2900
-Wire Wire Line
-	6150 3000 7750 3000
-Wire Wire Line
-	6150 3100 7750 3100
 Wire Bus Line
 	4100 2800 4100 3800
@@
 	7750 4750 7450 4750
 Wire Wire Line
-	7750 4850 7450 4850
-Wire Wire Line
 	7750 4950 7450 4950
 Wire Wire Line
+	7750 5050 7450 5050
+Wire Wire Line
 	6150 3300 6450 3300
 Wire Wire Line
@@
 Entry Wire Line
 	6450 4000 6550 4100
-Wire Bus Line
-	6550 3250 6550 4250
 Wire Wire Line
 	3800 2700 4850 2700
@@
 	4500 3800 4500 2800
 Wire Wire Line
-	7750 5050 7450 5050
-Wire Wire Line
 	7750 5150 7450 5150
+Wire Wire Line
+	7750 5250 7450 5250
 Entry Wire Line
 	7350 4850 7450 4750
 Entry Wire Line
-	7350 4950 7450 4850
-Entry Wire Line
 	7350 5050 7450 4950
 Entry Wire Line
 	7350 5150 7450 5050
+Entry Wire Line
+	7350 5250 7450 5150
 Entry Wire Line
 	4500 1900 4600 1800
 Text Label 7500 4750 0    60   ~ 0
 RESET_SPC
-Text Label 7500 4850 0    60   ~ 0
+Text Label 7500 4950 0    60   ~ 0
 /CS
-Text Label 7500 4950 0    60   ~ 0
+Text Label 7500 5050 0    60   ~ 0
 /RD
-Text Label 7500 5050 0    60   ~ 0
+Text Label 7500 5150 0    60   ~ 0
 /WR
 Wire Wire Line
@@
 Text Label 2300 3450 0    60   ~ 0
 /WR
-Text Label 7500 5150 0    60   ~ 0
+Text Label 7500 5250 0    60   ~ 0
 A0
 Entry Wire Line
+	7350 5550 7450 5450
+Entry Wire Line
 	7350 5350 7450 5250
-Entry Wire Line
-	7350 5250 7450 5150
-Text Label 7500 5250 0    60   ~ 0
+Text Label 7500 5450 0    60   ~ 0
 A1
 Wire Wire Line
-	7450 5250 7750 5250
-Entry Wire Line
-	7350 5550 7450 5450
-Wire Wire Line
 	7450 5450 7750 5450
-Text Label 7500 5450 0    60   ~ 0
+Entry Wire Line
+	7350 5650 7450 5550
+Wire Wire Line
+	7450 5550 7750 5550
+Text Label 7450 5650 0    60   ~ 0
 RESET
 Wire Bus Line
@@
 PC7
 Wire Wire Line
-	9650 4350 9950 4350
-Wire Wire Line
-	9650 4450 9950 4450
-Wire Wire Line
-	9650 4550 9950 4550
-Wire Wire Line
-	9650 4650 9950 4650
-Wire Wire Line
-	9650 4750 9950 4750
-Wire Wire Line
-	9650 4850 9950 4850
-Wire Wire Line
-	9650 4950 9950 4950
-Wire Wire Line
-	9650 5050 9950 5050
+	7400 3100 7750 3100
+Wire Wire Line
+	7400 3000 7750 3000
+Wire Wire Line
+	7400 2900 7750 2900
+Wire Wire Line
+	7400 2800 7750 2800
+Wire Wire Line
+	7400 2700 7750 2700
+Wire Wire Line
+	7400 2600 7750 2600
+Wire Wire Line
+	7400 2500 7750 2500
+Wire Wire Line
+	7400 2400 7750 2400
 Entry Wire Line
 	9950 4350 10050 4450
@@
 Wire Bus Line
 	10050 4300 10050 5350
-Text Label 9700 4350 0    60   ~ 0
+Text Label 7500 3100 0    60   ~ 0
 PC0
-Text Label 9700 4450 0    60   ~ 0
+Text Label 7500 3000 0    60   ~ 0
 PC1
-Text Label 9700 4550 0    60   ~ 0
+Text Label 7500 2900 0    60   ~ 0
 PC2
-Text Label 9700 4650 0    60   ~ 0
+Text Label 7500 2800 0    60   ~ 0
 PC3
-Text Label 9700 4750 0    60   ~ 0
+Text Label 7500 2700 0    60   ~ 0
 PC4
-Text Label 9700 4850 0    60   ~ 0
+Text Label 7500 2600 0    60   ~ 0
 PC5
-Text Label 9700 4950 0    60   ~ 0
+Text Label 7500 2500 0    60   ~ 0
 PC6
-Text Label 9700 5050 0    60   ~ 0
+Text Label 7500 2400 0    60   ~ 0
 PC7
 Text GLabel 10150 5350 2    60   Input ~ 0
-PC
+PA
 Wire Bus Line
 	10050 5350 10150 5350
@@
 Wire Wire Line
 	7750 3400 7500 3400
-Wire Wire Line
-	7750 3300 7600 3300
-Wire Wire Line
-	7600 3300 7600 3400
 Connection ~ 7600 3400
 Wire Wire Line
@@
 	9750 5450 9750 5350
 Connection ~ 9750 5350
-Wire Wire Line
-	6150 1500 7750 1500
 Entry Wire Line
 	7350 4450 7450 4350
@@
 Text Notes 8450 7650 0    60   ~ 12
 2015.06.26
+Wire Wire Line
+	6150 2400 6450 2400
+Wire Wire Line
+	6150 2500 6450 2500
+Wire Wire Line
+	6150 2600 6450 2600
+Wire Wire Line
+	6150 2700 6450 2700
+Wire Wire Line
+	6150 2800 6450 2800
+Wire Wire Line
+	6150 2900 6450 2900
+Wire Wire Line
+	6150 3000 6450 3000
+Wire Wire Line
+	6150 3100 6450 3100
+Entry Wire Line
+	6450 2400 6550 2500
+Entry Wire Line
+	6450 2500 6550 2600
+Entry Wire Line
+	6450 2600 6550 2700
+Entry Wire Line
+	6450 2700 6550 2800
+Entry Wire Line
+	6450 2800 6550 2900
+Entry Wire Line
+	6450 2900 6550 3000
+Entry Wire Line
+	6450 3000 6550 3100
+Entry Wire Line
+	6450 3100 6550 3200
+Text GLabel 6650 3200 2    60   Input ~ 0
+PB
+Wire Bus Line
+	6550 3250 6550 4250
+Wire Bus Line
+	6650 3200 6550 3200
+Wire Bus Line
+	6550 3200 6550 2400
+Wire Wire Line
+	6150 1500 6450 1500
+Wire Wire Line
+	6150 1600 6450 1600
+Wire Wire Line
+	6150 1700 6450 1700
+Wire Wire Line
+	6150 1800 6450 1800
+Wire Wire Line
+	6150 1900 6450 1900
+Wire Wire Line
+	6150 2000 6450 2000
+Wire Wire Line
+	6150 2100 6450 2100
+Wire Wire Line
+	6150 2200 6450 2200
+Entry Wire Line
+	6450 1500 6550 1600
+Entry Wire Line
+	6450 1600 6550 1700
+Entry Wire Line
+	6450 1700 6550 1800
+Entry Wire Line
+	6450 1800 6550 1900
+Entry Wire Line
+	6450 1900 6550 2000
+Entry Wire Line
+	6450 2000 6550 2100
+Entry Wire Line
+	6450 2100 6550 2200
+Entry Wire Line
+	6450 2200 6550 2300
+Text GLabel 7200 2300 0    60   Input ~ 0
+PB
+Wire Bus Line
+	6650 2300 6550 2300
+Wire Bus Line
+	6550 2300 6550 1500
+Text Label 6200 1500 0    60   ~ 0
+PA0
+Text Label 6200 1600 0    60   ~ 0
+PA1
+Text Label 6200 1700 0    60   ~ 0
+PA2
+Text Label 6200 1800 0    60   ~ 0
+PA3
+Text Label 6200 1900 0    60   ~ 0
+PA4
+Text Label 6200 2000 0    60   ~ 0
+PA5
+Text Label 6200 2100 0    60   ~ 0
+PA6
+Text Label 6200 2200 0    60   ~ 0
+PA7
+Text Label 6200 2400 0    60   ~ 0
+PB0
+Text Label 6200 2500 0    60   ~ 0
+PB1
+Text Label 6200 2600 0    60   ~ 0
+PB2
+Text Label 6200 2700 0    60   ~ 0
+PB3
+Text Label 6200 2800 0    60   ~ 0
+PB4
+Text Label 6200 2900 0    60   ~ 0
+PB5
+Text Label 6200 3000 0    60   ~ 0
+PB6
+Text Label 6200 3100 0    60   ~ 0
+PB7
+Wire Wire Line
+	7400 1500 7750 1500
+Wire Wire Line
+	7400 1600 7750 1600
+Wire Wire Line
+	7400 1700 7750 1700
+Wire Wire Line
+	7400 1800 7750 1800
+Wire Wire Line
+	7400 1900 7750 1900
+Wire Wire Line
+	7400 2000 7750 2000
+Wire Wire Line
+	7400 2100 7750 2100
+Wire Wire Line
+	7400 2200 7750 2200
+Entry Wire Line
+	7400 1500 7300 1600
+Entry Wire Line
+	7400 1600 7300 1700
+Entry Wire Line
+	7400 1700 7300 1800
+Entry Wire Line
+	7400 1800 7300 1900
+Entry Wire Line
+	7400 1900 7300 2000
+Entry Wire Line
+	7400 2000 7300 2100
+Entry Wire Line
+	7400 2100 7300 2200
+Entry Wire Line
+	7400 2200 7300 2300
+Text GLabel 6650 2300 2    60   Input ~ 0
+PA
+Wire Bus Line
+	7200 2300 7300 2300
+Wire Bus Line
+	7300 2300 7300 1500
+Text Label 7650 1500 2    60   ~ 0
+PB0
+Text Label 7650 1600 2    60   ~ 0
+PB1
+Text Label 7650 1700 2    60   ~ 0
+PB2
+Text Label 7650 1800 2    60   ~ 0
+PB3
+Text Label 7650 1900 2    60   ~ 0
+PB4
+Text Label 7650 2000 2    60   ~ 0
+PB5
+Text Label 7650 2100 2    60   ~ 0
+PB6
+Text Label 7650 2200 2    60   ~ 0
+PB7
+Text GLabel 7200 3200 0    60   Input ~ 0
+PC
+Entry Wire Line
+	7400 2400 7300 2500
+Entry Wire Line
+	7400 2500 7300 2600
+Entry Wire Line
+	7400 2600 7300 2700
+Entry Wire Line
+	7400 2700 7300 2800
+Entry Wire Line
+	7400 2800 7300 2900
+Entry Wire Line
+	7400 2900 7300 3000
+Entry Wire Line
+	7400 3000 7300 3100
+Entry Wire Line
+	7400 3100 7300 3200
+Wire Bus Line
+	7200 3200 7300 3200
+Wire Bus Line
+	7300 3200 7300 2400
+Wire Wire Line
+	9650 4350 9950 4350
+Wire Wire Line
+	9650 4450 9950 4450
+Wire Wire Line
+	9650 4550 9950 4550
+Wire Wire Line
+	9650 4650 9950 4650
+Wire Wire Line
+	9650 4750 9950 4750
+Wire Wire Line
+	9650 4850 9950 4850
+Wire Wire Line
+	9650 4950 9950 4950
+Wire Wire Line
+	9650 5050 9950 5050
+Text Label 9700 4350 0    60   ~ 0
+PA0
+Text Label 9700 4450 0    60   ~ 0
+PA1
+Text Label 9700 4550 0    60   ~ 0
+PA2
+Text Label 9700 4650 0    60   ~ 0
+PA3
+Text Label 9700 4750 0    60   ~ 0
+PA4
+Text Label 9700 4850 0    60   ~ 0
+PA5
+Text Label 9700 4950 0    60   ~ 0
+PA6
+Text Label 9700 5050 0    60   ~ 0
+PA7
 $EndSCHEMATC
