File: FDDuino.kicad/noname.kicad_pcb (KiCad board)
At the start: 2 copper layers, 12 parts, among them P1 RASPI_V2, P2 LS04, P3 LS04, P4 LS04, P5 LS04, P6 LS04, P7 MSX_SLOT, P8 LS04, U1 74LS74, U2 7400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

Commit message: Weekend works for FDDuino and MSXuino
Parts:
- removed U4: 7402, Housings_DIP:DIP-14_W7.62mm
- moved P1 41.9 mm to (175.3, 69.8), turned to 270 degrees
Connections:
- P2 pad 11: /MERQ -> /SLTSL
- U2 pad 10: (no net) -> Net-(U2-Pad10)
- U2 pad 11: Net-(U2-Pad11) -> Net-(U2-Pad10)
- U2 pad 2: /MERQ -> /SLTSL
- U2 pad 8: (no net) -> Net-(U1-Pad3)
- U2 pad 9: (no net) -> Net-(U2-Pad10)
