File: FDDuino.kicad/noname.sch (KiCad schematic (older format))
At the start: 12 parts, among them P1 RASPI_V2, P2 LS04, P3 LS04, P4 LS04, P5 LS04, P6 LS04, P7 MSX_SLOT, P8 LS04, U1 74LS74, U2 7400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

Commit message: Weekend works for FDDuino and MSXuino
Parts:
- removed U4: 7402, Housings_DIP:DIP-14_W7.62mm, symbol 7402
- added unit 3 of U2
Connections:
- net labels removed: /MERQ
- wire segments 189 -> 188
Changed lines of the file:
@@
 Text GLabel 4400 1100 0    60   Input ~ 0
 /IORQ
-Text GLabel 4400 1300 0    60   Input ~ 0
-/MERQ
 Text GLabel 4400 1600 0    60   Input ~ 0
 /WR
@@
 Text Notes 8150 7650 0    60   ~ 0
 2015.06.24
-Text GLabel 5400 2350 0    60   Input ~ 0
+Text GLabel 4400 1300 0    60   Input ~ 0
 /SLTSL
 Wire Wire Line
-	5650 1850 5650 2150
-Wire Wire Line
-	5400 2350 5650 2350
+	5650 1850 5650 2350
 Wire Wire Line
 	7550 3150 7700 3150
@@
 NoConn ~ 7300 4800
 $Comp
-L 7402 U4
-U 1 1 558BEC36
+L 7400 U2
+U 3 1 558D5F6F
 P 6250 2250
-F 0 "U4" H 6250 2300 60  0000 C CNN
-F 1 "7402" H 6300 2200 60  0000 C CNN
-F 2 "Housings_DIP:DIP-14_W7.62mm" H 6250 2250 60  0000 C CNN
+F 0 "U2" H 6250 2300 60  0000 C CNN
+F 1 "7400" H 6250 2150 60  0000 C CNN
+F 2 "" H 6250 2250 60  0000 C CNN
 F 3 "" H 6250 2250 60  0000 C CNN
-	1    6250 2250
-	1    0    0    -1
-$EndComp
+	3    6250 2250
+	1    0    0    -1
+$EndComp
