File: FDDuino.kicad/noname.sch (KiCad schematic (older format))
At the start: 11 parts, among them P1 RASPI_V2, P3 LS04, P5 LS04, P7 MSX_SLOT, U1 74LS74, U2 7400, U3 74F676

Commit message: FDDuino schematic update for correcting PIN number in Raspberry Pi GPIO
Parts:
- U4: renamed from U?; footprint (none) -> Housings_DIP:DIP-20_W7.62mm
- U5: renamed from U?; footprint (none) -> Housings_DIP:DIP-14_W7.62mm
- gave numbers to parts that had none: 1
Connections:
- net labels removed: A16
Changed lines of the file:
@@
 A12
 Text Label 8500 5100 0    60   ~ 0
+A13
+Text Label 8500 5200 0    60   ~ 0
 A14
-Text Label 8500 5200 0    60   ~ 0
+Text Label 8500 5300 0    60   ~ 0
 A15
-Text Label 8500 5300 0    60   ~ 0
-A16
 Text Label 9400 3250 0    60   ~ 0
 A9
@@
 Text GLabel 2350 2750 2    60   Input ~ 0
 G7
+Text GLabel 2300 3250 2    60   Input ~ 0
+G12
+Text GLabel 2300 3350 2    60   Input ~ 0
+G13
+Text GLabel 2300 3450 2    60   Input ~ 0
+G14
 Text GLabel 2300 3550 2    60   Input ~ 0
-G12
-Text GLabel 2300 3450 2    60   Input ~ 0
-G13
-Text GLabel 2300 3350 2    60   Input ~ 0
-G14
-Text GLabel 2300 3250 2    60   Input ~ 0
 G15
 Text GLabel 2300 3650 2    60   Input ~ 0
@@
 $EndComp
 $Comp
-L +5V #PWR011
+L +5V #PWR02
 U 1 1 558AEF5A
 P 1750 1550
-F 0 "#PWR011" H 1750 1400 50  0001 C CNN
+F 0 "#PWR02" H 1750 1400 50  0001 C CNN
 F 1 "+5V" H 1750 1690 50  0000 C CNN
 F 2 "" H 1750 1550 60  0000 C CNN
@@
 	1750 1550 1750 1800
 $Comp
-L GND #PWR012
+L GND #PWR03
 U 1 1 558B0DAF
 P 3200 2350
-F 0 "#PWR012" H 3200 2100 50  0001 C CNN
+F 0 "#PWR03" H 3200 2100 50  0001 C CNN
 F 1 "GND" H 3200 2200 50  0000 C CNN
 F 2 "" H 3200 2350 60  0000 C CNN
@@
 	3750 2250 3850 2250
 $Comp
-L +3.3V #PWR016
+L +3.3V #PWR04
 U 1 1 558B11D2
 P 2650 1950
-F 0 "#PWR016" H 2650 1800 50  0001 C CNN
+F 0 "#PWR04" H 2650 1800 50  0001 C CNN
 F 1 "+3.3V" H 2650 2090 50  0000 C CNN
 F 2 "" H 2650 1950 60  0000 C CNN
@@
 $EndComp
 $Comp
-L +5V #PWR017
+L +5V #PWR05
 U 1 1 558B701F
 P 5250 700
-F 0 "#PWR017" H 5250 550 50  0001 C CNN
+F 0 "#PWR05" H 5250 550 50  0001 C CNN
 F 1 "+5V" H 5250 840 50  0000 C CNN
 F 2 "" H 5250 700 60  0000 C CNN
@@
 $EndComp
 $Comp
-L GND #PWR018
+L GND #PWR06
 U 1 1 558B72A7
 P 5250 1850
-F 0 "#PWR018" H 5250 1600 50  0001 C CNN
+F 0 "#PWR06" H 5250 1600 50  0001 C CNN
 F 1 "GND" H 5250 1700 50  0000 C CNN
 F 2 "" H 5250 1850 60  0000 C CNN
@@
 $EndComp
 $Comp
-L +5V #PWR019
+L +5V #PWR07
 U 1 1 558B9971
 P 7800 1550
-F 0 "#PWR019" H 7800 1400 50  0001 C CNN
+F 0 "#PWR07" H 7800 1400 50  0001 C CNN
 F 1 "+5V" H 7800 1690 50  0000 C CNN
 F 2 "" H 7800 1550 60  0000 C CNN
@@
 $EndComp
 $Comp
-L GND #PWR020
+L GND #PWR08
 U 1 1 558B9998
 P 7800 2600
-F 0 "#PWR020" H 7800 2350 50  0001 C CNN
+F 0 "#PWR08" H 7800 2350 50  0001 C CNN
 F 1 "GND" H 7800 2450 50  0000 C CNN
 F 2 "" H 7800 2600 60  0000 C CNN
@@
 /WAIT_RESET
 $Comp
-L GND #PWR022
+L GND #PWR09
 U 1 1 558B9E5A
 P 7900 5600
-F 0 "#PWR022" H 7900 5350 50  0001 C CNN
+F 0 "#PWR09" H 7900 5350 50  0001 C CNN
 F 1 "GND" H 7900 5450 50  0000 C CNN
 F 2 "" H 7900 5600 60  0000 C CNN
@@
 	7900 3400 7900 3500
 $Comp
-L +5V #PWR023
+L +5V #PWR010
 U 1 1 558BA758
 P 9100 4750
-F 0 "#PWR023" H 9100 4600 50  0001 C CNN
+F 0 "#PWR010" H 9100 4600 50  0001 C CNN
 F 1 "+5V" H 9100 4890 50  0000 C CNN
 F 2 "" H 9100 4750 60  0000 C CNN
@@
 Connection ~ 9400 4750
 $Comp
-L GND #PWR024
+L GND #PWR011
 U 1 1 558BA923
 P 9400 4550
-F 0 "#PWR024" H 9400 4300 50  0001 C CNN
+F 0 "#PWR011" H 9400 4300 50  0001 C CNN
 F 1 "GND" H 9400 4400 50  0000 C CNN
 F 2 "" H 9400 4550 60  0000 C CNN
@@
 Connection ~ 9450 4550
 $Comp
-L +3.3V #PWR025
+L +3.3V #PWR012
 U 1 1 558BBE3A
 P 1450 1550
-F 0 "#PWR025" H 1450 1400 50  0001 C CNN
+F 0 "#PWR012" H 1450 1400 50  0001 C CNN
 F 1 "+3.3V" H 1450 1690 50  0000 C CNN
 F 2 "" H 1450 1550 60  0000 C CNN
@@
 	1450 1550 1450 1800
 $Comp
-L GND #PWR026
+L GND #PWR013
 U 1 1 558BC299
 P 1250 5250
-F 0 "#PWR026" H 1250 5000 50  0001 C CNN
+F 0 "#PWR013" H 1250 5000 50  0001 C CNN
 F 1 "GND" H 1250 5100 50  0000 C CNN
 F 2 "" H 1250 5250 60  0000 C CNN
@@
 	3750 2150 3950 2150
 $Comp
-L GND #PWR027
+L GND #PWR014
 U 1 1 558BBBCD
 P 7150 4200
-F 0 "#PWR027" H 7150 3950 50  0001 C CNN
+F 0 "#PWR014" H 7150 3950 50  0001 C CNN
 F 1 "GND" H 7150 4050 50  0000 C CNN
 F 2 "" H 7150 4200 60  0000 C CNN
@@
 $EndComp
 $Comp
-L 74LS245 U?
+L 74LS245 U4
 U 1 1 55927034
 P 3850 5000
-F 0 "U?" H 3950 5575 60  0000 L BNN
+F 0 "U4" H 3950 5575 60  0000 L BNN
 F 1 "74LS245" H 3900 4425 60  0000 L TNN
-F 2 "" H 3850 5000 60  0000 C CNN
+F 2 "Housings_DIP:DIP-20_W7.62mm" H 3850 5000 60  0000 C CNN
 F 3 "" H 3850 5000 60  0000 C CNN
 	1    3850 5000
@@
 	4800 6000 4800 4750
 $Comp
-L +3.3V #PWR?
+L +3.3V #PWR015
 U 1 1 55929288
 P 7900 3400
-F 0 "#PWR?" H 7900 3250 50  0001 C CNN
+F 0 "#PWR015" H 7900 3250 50  0001 C CNN
 F 1 "+3.3V" H 7900 3540 50  0000 C CNN
 F 2 "" H 7900 3400 60  0000 C CNN
@@
 	3750 3400 4000 3400
 $Comp
-L GND #PWR?
+L GND #PWR016
 U 1 1 5592B35A
 P 3750 3200
-F 0 "#PWR?" H 3750 2950 50  0001 C CNN
+F 0 "#PWR016" H 3750 2950 50  0001 C CNN
 F 1 "GND" H 3750 3050 50  0000 C CNN
 F 2 "" H 3750 3200 60  0000 C CNN
@@
 Connection ~ 3850 2250
 $Comp
-L GND #PWR?
+L GND #PWR017
 U 1 1 5592B4ED
 P 3150 3200
-F 0 "#PWR?" H 3150 2950 50  0001 C CNN
+F 0 "#PWR017" H 3150 2950 50  0001 C CNN
 F 1 "GND" H 3150 3050 50  0000 C CNN
 F 2 "" H 3150 3200 60  0000 C CNN
@@
 $EndComp
 $Comp
-L +5V #PWR?
+L +5V #PWR018
 U 1 1 5592B75B
 P 3850 1950
-F 0 "#PWR?" H 3850 1800 50  0001 C CNN
+F 0 "#PWR018" H 3850 1800 50  0001 C CNN
 F 1 "+5V" H 3850 2090 50  0000 C CNN
 F 2 "" H 3850 1950 60  0000 C CNN
@@
 Connection ~ 2650 3700
 $Comp
-L GND #PWR?
+L GND #PWR019
 U 1 1 5592BAAA
 P 4550 4500
-F 0 "#PWR?" H 4550 4250 50  0001 C CNN
+F 0 "#PWR019" H 4550 4250 50  0001 C CNN
 F 1 "GND" H 4550 4350 50  0000 C CNN
 F 2 "" H 4550 4500 60  0000 C CNN
@@
 	6750 4150 6750 4400
 $Comp
-L 74LS00 U?
+L 74LS00 U5
 U 1 1 5592E601
 P 5400 2750
-F 0 "U?" H 5400 2800 60  0000 C CNN
+F 0 "U5" H 5400 2800 60  0000 C CNN
 F 1 "74LS00" H 5400 2650 60  0000 C CNN
-F 2 "" H 5400 2750 60  0000 C CNN
+F 2 "Housings_DIP:DIP-14_W7.62mm" H 5400 2750 60  0000 C CNN
 F 3 "" H 5400 2750 60  0000 C CNN
 	1    5400 2750
@@
 $EndComp
 $Comp
-L 74LS00 U?
+L 74LS00 U5
 U 2 1 5592E787
 P 5400 3250
-F 0 "U?" H 5400 3300 60  0000 C CNN
+F 0 "U5" H 5400 3300 60  0000 C CNN
 F 1 "74LS00" H 5400 3150 60  0000 C CNN
 F 2 "" H 5400 3250 60  0000 C CNN
@@
 $EndComp
 $Comp
-L 74LS00 U?
+L 74LS00 U5
 U 3 1 5592E7D9
 P 6600 3000
-F 0 "U?" H 6600 3050 60  0000 C CNN
+F 0 "U5" H 6600 3050 60  0000 C CNN
 F 1 "74LS00" H 6600 2900 60  0000 C CNN
 F 2 "" H 6600 3000 60  0000 C CNN
@@
 	7200 2400 7200 3000
 $Comp
-L +5V #PWR?
+L +5V #PWR020
 U 1 1 55930E0B
 P 5200 2450
-F 0 "#PWR?" H 5200 2300 50  0001 C CNN
+F 0 "#PWR020" H 5200 2300 50  0001 C CNN
 F 1 "+5V" H 5200 2590 50  0000 C CNN
 F 2 "" H 5200 2450 60  0000 C CNN
@@
 $EndComp
 $Comp
-L GND #PWR?
+L GND #PWR021
 U 1 1 55930E58
 P 5200 3500
-F 0 "#PWR?" H 5200 3250 50  0001 C CNN
+F 0 "#PWR021" H 5200 3250 50  0001 C CNN
 F 1 "GND" H 5200 3350 50  0000 C CNN
 F 2 "" H 5200 3500 60  0000 C CNN
