File: FDDuino.kicad/$Z80Raspi.sch (KiCad schematic (older format))
At the start: 3 parts, among them P1 RASPI_V2, U1 74F676, U2 Z80CPU

Commit message: FDDuino update
Parts:
- U1: footprint Housings_DIP:DIP-40_W15.24mm -> Housings_DIP:DIP-24_W10.16mm
Changed lines of the file:
@@
 F 0 "U1" H 4050 4400 50  0000 L CNN
 F 1 "74F676" H 4650 4400 50  0000 L CNN
-F 2 "Housings_DIP:DIP-40_W15.24mm" H 4500 3600 60  0000 C CNN
+F 2 "Housings_DIP:DIP-24_W10.16mm" H 4500 3600 60  0000 C CNN
 F 3 "" H 4500 3600 60  0000 C CNN
 	1    4500 3600
