File: FDDuino.kicad/_autosave-Z80Raspi.kicad_pcb (KiCad board)
At the start: 2 copper layers, 3 parts, among them P1 RASPI_V2, U1 74F676, U2 Z80CPU

Commit message: FDDuino update
Parts:
- U1, U2: moved to B.Cu
- moved U1 47.4 mm to (127.6, 127.6)
- moved P1 38.7 mm to (121.9, 89.5)
- moved U2 22.9 mm to (156.2, 89.5), turned to 180 degrees
